File: hardware/simon-game.sch (KiCad schematic (older format))
At the start: 17 parts, among them SW1 SW_Push, SW2 SW_Push, SW3 SW_Push, SW4 SW_Push, U1 ATtiny402-SS

Commit message: Finished PCB
Parts:
- removed SW4: SW_Push, Button_Switch_THT:SW_PUSH_6mm, symbol Switch:SW_Push
- added J?: Conn_01x03_Male, symbol Connector:Conn_01x03_Male
- added SW4: TACTILE_SW_4Pin, ingus_electromechanics:6x6_SPST, symbol raksts:TACTILE_SW_4Pin
- BZ1: footprint Buzzer_Beeper:Buzzer_12x9.5RM7.6 -> ingus_electromechanics:Beeper_12xx
- C1: footprint Capacitor_THT:C_Disc_D4.3mm_W1.9mm_P5.00mm -> janis:CE-2mm54
- R1, R2, R3, R4, R5: footprint Resistor_THT:R_Axial_DIN0207_L6.3mm_D2.5mm_P7.62mm_Horizontal -> janis:R_W8_THT_Hor
- SW1, SW2, SW3: footprint Button_Switch_THT:SW_PUSH_6mm -> ingus_electromechanics:6x6_SPST; symbol Switch:SW_Push -> raksts:TACTILE_SW_4Pin
Connections:
- net GND: now also SW1.3, SW1.4, SW2.3, SW2.4, SW3.3, SW3.4, J?.3 (Pin_3), SW4.3, SW4.4; no longer SW1.2, SW2.2, SW3.2
- net RESET_UPDI: now also J?.2 (Pin_2)
- net at BAT1.1, BZ1.1 (-), C1.1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: now also J?.1 (Pin_1)
- net at D1.1 (K), SW1.1, U1.3 (PA7): now also SW1.2
- net at D4.1 (K), U1.4 (PA1): now also SW4.1, SW4.2
- net at D3.1 (K), SW3.1, U1.5 (PA2): now also SW3.2
- net at D2.1 (K), SW2.1, U1.7 (PA3): now also SW2.2
Changed lines of the file:
@@
 F 0 "C1" H 4792 3146 50  0000 L CNN
 F 1 "0.1uF" H 4792 3055 50  0000 L CNN
-F 2 "Capacitor_THT:C_Disc_D4.3mm_W1.9mm_P5.00mm" H 4700 3100 50  0001 C CNN
+F 2 "janis:CE-2mm54" H 4700 3100 50  0001 C CNN
 F 3 "~" H 4700 3100 50  0001 C CNN
 	1    4700 3100
@@
 	1    0    0    -1
 $EndComp
-Wire Wire Line
-	6300 3400 6800 3400
 Text Label 6800 3400 2    50   ~ 0
 RESET_UPDI
@@
 F 0 "R1" H 8359 3046 50  0000 L CNN
 F 1 "220" H 8359 2955 50  0000 L CNN
-F 2 "Resistor_THT:R_Axial_DIN0207_L6.3mm_D2.5mm_P7.62mm_Horizontal" H 8300 3000 50  0001 C CNN
+F 2 "janis:R_W8_THT_Hor" H 8300 3000 50  0001 C CNN
 F 3 "~" H 8300 3000 50  0001 C CNN
 	1    8300 3000
@@
 	8300 3200 8300 3100
 $Comp
-L Switch:SW_Push SW1
+L raksts:TACTILE_SW_4Pin SW1
 U 1 1 5DB94A81
-P 8300 4200
-F 0 "SW1" V 8254 4348 50  0000 L CNN
-F 1 "SW_Push" V 8345 4348 50  0000 L CNN
-F 2 "Button_Switch_THT:SW_PUSH_6mm" H 8300 4400 50  0001 C CNN
-F 3 "~" H 8300 4400 50  0001 C CNN
-	1    8300 4200
+P 8400 4300
+F 0 "SW1" V 8354 4448 50  0000 L CNN
+F 1 "SW_Push" V 8445 4448 50  0000 L CNN
+F 2 "ingus_electromechanics:6x6_SPST" H 8400 4500 50  0001 C CNN
+F 3 "~" H 8400 4500 50  0001 C CNN
+	1    8400 4300
 	0    1    1    0
 $EndComp
@@
 Wire Wire Line
 	8300 3400 8300 3900
-Wire Wire Line
-	8300 4400 8300 4500
 $Comp
 L power:GND #PWR0103
 U 1 1 5DB97DA0
-P 8300 4500
-F 0 "#PWR0103" H 8300 4250 50  0001 C CNN
-F 1 "GND" H 8305 4327 50  0000 C CNN
-F 2 "" H 8300 4500 50  0001 C CNN
-F 3 "" H 8300 4500 50  0001 C CNN
-	1    8300 4500
+P 8300 4800
+F 0 "#PWR0103" H 8300 4550 50  0001 C CNN
+F 1 "GND" H 8305 4627 50  0000 C CNN
+F 2 "" H 8300 4800 50  0001 C CNN
+F 3 "" H 8300 4800 50  0001 C CNN
+	1    8300 4800
 	1    0    0    -1
 $EndComp
@@
 F 0 "R3" H 8859 3046 50  0000 L CNN
 F 1 "220" H 8859 2955 50  0000 L CNN
-F 2 "Resistor_THT:R_Axial_DIN0207_L6.3mm_D2.5mm_P7.62mm_Horizontal" H 8800 3000 50  0001 C CNN
+F 2 "janis:R_W8_THT_Hor" H 8800 3000 50  0001 C CNN
 F 3 "~" H 8800 3000 50  0001 C CNN
 	1    8800 3000
@@
 	8800 3200 8800 3100
 $Comp
-L Switch:SW_Push SW2
+L raksts:TACTILE_SW_4Pin SW2
 U 1 1 5DB9A895
-P 8800 4200
-F 0 "SW2" V 8754 4348 50  0000 L CNN
-F 1 "SW_Push" V 8845 4348 50  0000 L CNN
-F 2 "Button_Switch_THT:SW_PUSH_6mm" H 8800 4400 50  0001 C CNN
-F 3 "~" H 8800 4400 50  0001 C CNN
-	1    8800 4200
+P 8900 4300
+F 0 "SW2" V 8854 4448 50  0000 L CNN
+F 1 "SW_Push" V 8945 4448 50  0000 L CNN
+F 2 "ingus_electromechanics:6x6_SPST" H 8900 4500 50  0001 C CNN
+F 3 "~" H 8900 4500 50  0001 C CNN
+	1    8900 4300
 	0    1    1    0
 $EndComp
 Wire Wire Line
 	8800 2900 8800 2800
-Wire Wire Line
-	8800 4400 8800 4500
 $Comp
 L power:GND #PWR0104
 U 1 1 5DB9A8A2
-P 8800 4500
-F 0 "#PWR0104" H 8800 4250 50  0001 C CNN
-F 1 "GND" H 8805 4327 50  0000 C CNN
-F 2 "" H 8800 4500 50  0001 C CNN
-F 3 "" H 8800 4500 50  0001 C CNN
-	1    8800 4500
+P 8800 4800
+F 0 "#PWR0104" H 8800 4550 50  0001 C CNN
+F 1 "GND" H 8805 4627 50  0000 C CNN
+F 2 "" H 8800 4800 50  0001 C CNN
+F 3 "" H 8800 4800 50  0001 C CNN
+	1    8800 4800
 	1    0    0    -1
 $EndComp
@@
 F 0 "R4" H 9359 3046 50  0000 L CNN
 F 1 "220" H 9359 2955 50  0000 L CNN
-F 2 "Resistor_THT:R_Axial_DIN0207_L6.3mm_D2.5mm_P7.62mm_Horizontal" H 9300 3000 50  0001 C CNN
+F 2 "janis:R_W8_THT_Hor" H 9300 3000 50  0001 C CNN
 F 3 "~" H 9300 3000 50  0001 C CNN
 	1    9300 3000
@@
 Wire Wire Line
 	9300 3200 9300 3100
-$Comp
-L Switch:SW_Push SW3
-U 1 1 5DBA05D3
-P 9300 4200
-F 0 "SW3" V 9254 4348 50  0000 L CNN
-F 1 "SW_Push" V 9345 4348 50  0000 L CNN
-F 2 "Button_Switch_THT:SW_PUSH_6mm" H 9300 4400 50  0001 C CNN
-F 3 "~" H 9300 4400 50  0001 C CNN
-	1    9300 4200
-	0    1    1    0
-$EndComp
 Wire Wire Line
 	9300 2900 9300 2800
-Wire Wire Line
-	9300 4400 9300 4500
 $Comp
 L power:GND #PWR0105
 U 1 1 5DBA05DB
-P 9300 4500
-F 0 "#PWR0105" H 9300 4250 50  0001 C CNN
-F 1 "GND" H 9305 4327 50  0000 C CNN
-F 2 "" H 9300 4500 50  0001 C CNN
-F 3 "" H 9300 4500 50  0001 C CNN
-	1    9300 4500
+P 9300 4800
+F 0 "#PWR0105" H 9300 4550 50  0001 C CNN
+F 1 "GND" H 9305 4627 50  0000 C CNN
+F 2 "" H 9300 4800 50  0001 C CNN
+F 3 "" H 9300 4800 50  0001 C CNN
+	1    9300 4800
 	1    0    0    -1
 $EndComp
@@
 F 0 "R5" H 9859 3046 50  0000 L CNN
 F 1 "220" H 9859 2955 50  0000 L CNN
-F 2 "Resistor_THT:R_Axial_DIN0207_L6.3mm_D2.5mm_P7.62mm_Horizontal" H 9800 3000 50  0001 C CNN
+F 2 "janis:R_W8_THT_Hor" H 9800 3000 50  0001 C CNN
 F 3 "~" H 9800 3000 50  0001 C CNN
 	1    9800 3000
@@
 Wire Wire Line
 	9800 3200 9800 3100
-$Comp
-L Switch:SW_Push SW4
-U 1 1 5DBA1900
-P 9800 4200
-F 0 "SW4" V 9754 4348 50  0000 L CNN
-F 1 "SW_Push" V 9845 4348 50  0000 L CNN
-F 2 "Button_Switch_THT:SW_PUSH_6mm" H 9800 4400 50  0001 C CNN
-F 3 "~" H 9800 4400 50  0001 C CNN
-	1    9800 4200
-	0    1    1    0
-$EndComp
 Wire Wire Line
 	9800 2900 9800 2800
 Wire Wire Line
-	9800 4400 9800 4500
+	9800 4600 9800 4700
 $Comp
 L power:GND #PWR0106
 U 1 1 5DBA1908
-P 9800 4500
-F 0 "#PWR0106" H 9800 4250 50  0001 C CNN
-F 1 "GND" H 9805 4327 50  0000 C CNN
-F 2 "" H 9800 4500 50  0001 C CNN
-F 3 "" H 9800 4500 50  0001 C CNN
-	1    9800 4500
+P 9800 4800
+F 0 "#PWR0106" H 9800 4550 50  0001 C CNN
+F 1 "GND" H 9805 4627 50  0000 C CNN
+F 2 "" H 9800 4800 50  0001 C CNN
+F 3 "" H 9800 4800 50  0001 C CNN
+	1    9800 4800
 	1    0    0    -1
 $EndComp
@@
 Connection ~ 8800 3700
 Wire Wire Line
-	8800 3700 8800 4000
-Wire Wire Line
 	6300 3600 9300 3600
 Connection ~ 9300 3600
 Wire Wire Line
-	9300 3600 9300 4000
+	9300 3600 9300 3900
 Wire Wire Line
 	6300 3500 9800 3500
 Connection ~ 9800 3500
 Wire Wire Line
-	9800 3500 9800 4000
+	9800 3500 9800 3900
 $Comp
 L Device:Buzzer BZ1
@@
 F 0 "BZ1" H 7852 3129 50  0000 L CNN
 F 1 "Buzzer" H 7852 3038 50  0000 L CNN
-F 2 "Buzzer_Beeper:Buzzer_12x9.5RM7.6" V 7675 3200 50  0001 C CNN
+F 2 "ingus_electromechanics:Beeper_12xx" V 7675 3200 50  0001 C CNN
 F 3 "~" V 7675 3200 50  0001 C CNN
 	1    7700 3100
@@
 F 0 "R2" H 7359 3146 50  0000 L CNN
 F 1 "10k" H 7359 3055 50  0000 L CNN
-F 2 "Resistor_THT:R_Axial_DIN0207_L6.3mm_D2.5mm_P7.62mm_Horizontal" H 7300 3100 50  0001 C CNN
+F 2 "janis:R_W8_THT_Hor" H 7300 3100 50  0001 C CNN
 F 3 "~" H 7300 3100 50  0001 C CNN
 	1    7300 3100
@@
 $EndComp
 Wire Wire Line
-	5700 2800 7300 2800
+	5700 2800 6600 2800
 Wire Wire Line
 	7600 3000 7500 3000
@@
 	6300 3800 7300 3800
 Connection ~ 7300 3300
+$Comp
+L raksts:TACTILE_SW_4Pin SW4
+U 1 1 5DC5D6E3
+P 9900 4300
+F 0 "SW4" V 9854 4418 50  0000 L CNN
+F 1 "TACTILE_SW_4Pin" V 9945 4418 50  0000 L CNN
+F 2 "ingus_electromechanics:6x6_SPST" H 9900 4300 50  0001 C CNN
+F 3 "" H 9900 4300 50  0000 C CNN
+	1    9900 4300
+	0    1    1    0
+$EndComp
+Wire Wire Line
+	9800 3900 9900 3900
+Wire Wire Line
+	9900 3900 9900 4000
+Connection ~ 9800 3900
+Wire Wire Line
+	9800 3900 9800 4000
+Wire Wire Line
+	9900 4600 9900 4700
+Wire Wire Line
+	9900 4700 9800 4700
+Wire Wire Line
+	9800 4800 9800 4700
+Connection ~ 9800 4700
+Wire Wire Line
+	8800 3700 8800 3900
+$Comp
+L raksts:TACTILE_SW_4Pin SW3
+U 1 1 5DBA05D3
+P 9400 4300
+F 0 "SW3" V 9354 4448 50  0000 L CNN
+F 1 "SW_Push" V 9445 4448 50  0000 L CNN
+F 2 "ingus_electromechanics:6x6_SPST" H 9400 4500 50  0001 C CNN
+F 3 "~" H 9400 4500 50  0001 C CNN
+	1    9400 4300
+	0    1    1    0
+$EndComp
+Wire Wire Line
+	9300 3900 9400 3900
+Wire Wire Line
+	9400 3900 9400 4000
+Connection ~ 9300 3900
+Wire Wire Line
+	9300 3900 9300 4000
+Wire Wire Line
+	8800 3900 8900 3900
+Wire Wire Line
+	8900 3900 8900 4000
+Connection ~ 8800 3900
+Wire Wire Line
+	8800 3900 8800 4000
+Wire Wire Line
+	8300 3900 8400 3900
+Wire Wire Line
+	8400 3900 8400 4000
+Wire Wire Line
+	8300 4600 8300 4700
+Wire Wire Line
+	8300 4700 8400 4700
+Wire Wire Line
+	8400 4700 8400 4600
+Wire Wire Line
+	8800 4600 8800 4700
+Wire Wire Line
+	8800 4700 8900 4700
+Wire Wire Line
+	8900 4700 8900 4600
+Wire Wire Line
+	9300 4600 9300 4700
+Wire Wire Line
+	9300 4700 9400 4700
+Wire Wire Line
+	9400 4700 9400 4600
+Wire Wire Line
+	9300 4800 9300 4700
+Connection ~ 9300 4700
+Wire Wire Line
+	8800 4800 8800 4700
+Connection ~ 8800 4700
+Wire Wire Line
+	8300 4800 8300 4700
+Connection ~ 8300 4700
+$Comp
+L Connector:Conn_01x03_Male J?
+U 1 1 5DC7CE07
+P 6100 2100
+F 0 "J?" H 6208 2381 50  0000 C CNN
+F 1 "Conn_01x03_Male" H 6208 2290 50  0000 C CNN
+F 2 "" H 6100 2100 50  0001 C CNN
+F 3 "~" H 6100 2100 50  0001 C CNN
+	1    6100 2100
+	1    0    0    -1
+$EndComp
+Wire Wire Line
+	6300 2000 6600 2000
+Wire Wire Line
+	6600 2000 6600 2800
+Connection ~ 6600 2800
+Wire Wire Line
+	6600 2800 7300 2800
+Wire Wire Line
+	6300 2100 6900 2100
+Wire Wire Line
+	6900 2100 6900 3400
+Wire Wire Line
+	6300 3400 6900 3400
+Wire Wire Line
+	6300 2200 6400 2200
+Wire Wire Line
+	6400 2200 6400 2300
+$Comp
+L power:GND #PWR?
+U 1 1 5DC82D95
+P 6400 2300
+F 0 "#PWR?" H 6400 2050 50  0001 C CNN
+F 1 "GND" H 6405 2127 50  0000 C CNN
+F 2 "" H 6400 2300 50  0001 C CNN
+F 3 "" H 6400 2300 50  0001 C CNN
+	1    6400 2300
+	1    0    0    -1
+$EndComp
+Connection ~ 6400 2200
 $EndSCHEMATC

Commit message: Fixed battery orientation
Parts:
- J1: renamed from J?; footprint (none) -> Connector_PinSocket_2.54mm:PinSocket_1x03_P2.54mm_Vertical
Changed lines of the file:
@@
 Connection ~ 8300 4700
 $Comp
-L Connector:Conn_01x03_Male J?
+L Connector:Conn_01x03_Male J1
 U 1 1 5DC7CE07
 P 6100 2100
-F 0 "J?" H 6208 2381 50  0000 C CNN
+F 0 "J1" H 6208 2381 50  0000 C CNN
 F 1 "Conn_01x03_Male" H 6208 2290 50  0000 C CNN
-F 2 "" H 6100 2100 50  0001 C CNN
+F 2 "Connector_PinSocket_2.54mm:PinSocket_1x03_P2.54mm_Vertical" H 6100 2100 50  0001 C CNN
 F 3 "~" H 6100 2100 50  0001 C CNN
 	1    6100 2100
@@
 	6400 2200 6400 2300
 $Comp
-L power:GND #PWR?
+L power:GND #PWR0107
 U 1 1 5DC82D95
 P 6400 2300
-F 0 "#PWR?" H 6400 2050 50  0001 C CNN
+F 0 "#PWR0107" H 6400 2050 50  0001 C CNN
 F 1 "GND" H 6405 2127 50  0000 C CNN
 F 2 "" H 6400 2300 50  0001 C CNN

Commit message: New STM32G030 based hardware
Parts:
- removed J1: Conn_01x03_Male, Connector_PinSocket_2.54mm:PinSocket_1x03_P2.54mm_Vertical, symbol Connector:Conn_01x03_Male
- removed U1: ATtiny402-SS, Package_SO:SOIC-8_3.9x4.9mm_P1.27mm, symbol MCU_Microchip_ATtiny:ATtiny402-SS
- added DD1: STM32G030Fxx, Package_SO:TSSOP-20_4.4x6.5mm_P0.65mm, symbol janis:STM32G030Fxx
- added J1: Conn_01x05, Connector_PinHeader_2.54mm:PinHeader_1x05_P2.54mm_Vertical, symbol Connector_Generic:Conn_01x05
- added J2, J3: Conn_01x01, TestPoint:TestPoint_Pad_D2.0mm, symbol Connector_Generic:Conn_01x01
- BAT1: symbol electromechanics_ingus:CR2032_V -> simon-game-rescue:CR2032_V-electromechanics_ingus
Connections:
- net BUZZER: now also DD1.1 (PB7/PB8)
- net GND: now also D1.1 (K), D2.1 (K), D3.1 (K), D4.1 (K), DD1.5 (VSS/VSSA), J1.1 (Pin_1)
- net VBAT: now reaches BAT1.1, BZ1.1 (-), C1.1, R2.1
- net VBAT: now also DD1.4 (VDD/VDDA), J1.2 (Pin_2); no longer R1.1, R3.1, R4.1, R5.1
- net GREEN: now reaches SW1.1, SW1.2
- net GREEN: now also DD1.7 (PA0); no longer D1.1 (K)
- net YELLOW: now reaches SW4.1, SW4.2
- net YELLOW: now also DD1.9 (PA2); no longer D4.1 (K)
- net BLUE: now reaches SW3.1, SW3.2
- net BLUE: now also DD1.11 (PA4); no longer D3.1 (K)
- net RED: now reaches SW2.1, SW2.2
- net RED: now also DD1.20 (PB3/PB4/PB5/PB6); no longer D2.1 (K)
- new net: DD1.16 ([PA9]PA11), J2.1 (Pin_1)
- new net: DD1.17 ([PA10]PA12), J3.1 (Pin_1)
- new net LED_BLUE: DD1.12 (PA5), R4.1
- new net LED_GREEN: DD1.8 (PA1), R1.1
- new net LED_RED: DD1.14 (PA7), R3.1
- new net LED_YELLOW: DD1.10 (PA3), R5.1
- new net RESET: DD1.6 (NRST), J1.5 (Pin_5)
- new net SWCLK: DD1.19 (SWCLK/PA14-BOOT0/PA15), J1.4 (Pin_4)
- new net SWDIO: DD1.18 (SWDIO/PA13), J1.3 (Pin_3)
Other:
- moved on the sheet: BAT1, C1, D1, D2, D3, D4, R1, R3, R4, R5
